File: hardware/slcan.kicad_pcb (KiCad board)
At the start: 0 parts

Commit message: V1.0
Parts:
- added C1: 100n, Capacitor_SMD:C_0402_1005Metric, F.Cu at (134.4, 91.6)
- added C2: 100n, Capacitor_SMD:C_0402_1005Metric, F.Cu at (134.5, 101.1)
- added C3: 100n, Capacitor_SMD:C_0402_1005Metric, F.Cu at (145.9, 93.8)
- added C4: 22u, Capacitor_SMD:C_0402_1005Metric, F.Cu at (145.9, 92.8)
- added C5: 20p, Capacitor_SMD:C_0402_1005Metric, F.Cu at (149.2, 99.4)
- added C6: 20p, Capacitor_SMD:C_0402_1005Metric, F.Cu at (146.2, 102.8)
- added C7: 100n, Capacitor_SMD:C_0402_1005Metric, F.Cu at (137.1, 85.2)
- added D1: NUP2105L, Package_TO_SOT_SMD:SOT-23, F.Cu at (144.7, 85.8)
- added J1: 002, put_on_edge:on_edge_2x05_device, F.Cu at (127.4, 88.9)
- added J2: 025, put_on_edge:on_edge_2x05_host, F.Cu at (152.4, 88.9)
- added JP1: Jumper_2_Open, Connector_PinHeader_2.54mm:PinHeader_1x02_P2.54mm_Vertical, F.Cu at (138.3, 87.7)
- added JP2: Jumper_2_Open, Connector_PinHeader_2.54mm:PinHeader_1x02_P2.54mm_Vertical, F.Cu at (138.3, 82.8)
- added R1: 60, Resistor_SMD:R_0603_1608Metric, F.Cu at (135.4, 87.0)
- added R2: 60, Resistor_SMD:R_0603_1608Metric, F.Cu at (135.4, 83.7)
- added TP1: TXCAN, TestPoint:TestPoint_THTPad_D1.0mm_Drill0.5mm, F.Cu at (141.8, 102.9)
- added TP2: RXCAN, TestPoint:TestPoint_THTPad_D1.0mm_Drill0.5mm, F.Cu at (139.3, 102.9)
- added TP3: CANH, TestPoint:TestPoint_THTPad_D1.0mm_Drill0.5mm, F.Cu at (143.7, 89.1)
- added TP4: CANL, TestPoint:TestPoint_THTPad_D1.0mm_Drill0.5mm, F.Cu at (143.7, 82.2)
- added TP5: 20MHz, TestPoint:TestPoint_THTPad_D1.0mm_Drill0.5mm, F.Cu at (146.3, 97.8)
- added U1: MCP251863, Package_SO:SSOP-28_5.3x10.2mm_P0.65mm, F.Cu at (139.8, 96.3)
- added Y1: 20MHz, Crystal:Crystal_SMD_3225-4Pin_3.2x2.5mm, F.Cu at (148.8, 101.6)
Routing:
- net /can_to_spi_MCP25xx/CANL: track 0.00 -> 30.7 mm
- net /can_to_spi_MCP25xx/CANH: track 0.00 -> 23.3 mm
- net Net-(U1-RXCAN): track 0.00 -> 22.9 mm
- net /can_to_spi_MCP25xx/~{INT0}: track 0.00 -> 21.5 mm
- net /can_to_spi_MCP25xx/SCK: track 0.00 -> 19.4 mm
- net /can_to_spi_MCP25xx/~{CS}: track 0.00 -> 18.0 mm, vias 0 -> 1
- net GND: track 0.00 -> 17.4 mm, vias 0 -> 36
- net Net-(U1-TXCAN): track 0.00 -> 14.2 mm
- net /can_to_spi_MCP25xx/~{INT1}: track 0.00 -> 11.9 mm, vias 0 -> 1
- net /can_to_spi_MCP25xx/MOSI: track 0.00 -> 11.9 mm
- net /can_to_spi_MCP25xx/MISO: track 0.00 -> 10.8 mm
- net +3V3: track 0.00 -> 9.85 mm, vias 0 -> 4
- net +5V: track 0.00 -> 8.97 mm, vias 0 -> 1
- net /can_to_spi_MCP25xx/OSC1: track 0.00 -> 8.73 mm
- net /can_to_spi_MCP25xx/OSC2: track 0.00 -> 8.23 mm
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- added copper zone on In2.Cu, net +3V3
- added copper zone on B.Cu, net +5V
- added copper zone on F.Cu, net GND
- added copper zone on In1.Cu, net GND
Other:
- board outline added: 25 x 25 mm
- copper layers 0 -> 4
- board text added: "CAN FD"
- board text added: "V1.0"
